File: CP2104.sch (KiCad schematic (older format))
At the start: 8 parts, among them J7 USB_B_Mini, U4 CP2104

Commit message: update,
Parts:
- gave numbers to parts that had none: 1
Changed lines of the file:
@@
 $EndComp
 $Comp
-L taobao-sd:SD_1N4001_M1 D?
+L taobao-sd:SD_1N4001_M1 D5
 U 1 1 5C0DACA6
 P 3750 2550
-F 0 "D?" V 3700 2650 50  0000 L CNN
+F 0 "D5" V 3700 2650 50  0000 L CNN
 F 1 "SD_1N4001_M1" V 3750 2650 50  0000 L CNN
 F 2 "w_smd_diode:do214ac" V 3750 2550 50  0001 C CNN
