File: AMS1117-3.3.sch (KiCad schematic (older format))
At the start: 7 parts, among them J5 Conn_01x03, U2 AMS1117-3.3

Commit message: update,
Parts:
- added JP? (x2): Jumper_NO_Small, symbol Device:Jumper_NO_Small
Connections:
- net +3V3: now also JP?.1; no longer C8.1, C9.1, U2.2 (VO)
- net +5V: no longer names the net of C7.1, U2.3 (VI)
- net +5V: now also JP?.2
- new net: C8.1, C9.1, JP?.2, U2.2 (VO)
- new net VIN: JP?.1
Other:
- moved on the sheet: J5
Changed lines of the file:
@@
 $EndComp
-Wire Wire Line
-	1350 1650 1350 1800
-Wire Wire Line
-	1350 1800 2050 1800
-Wire Wire Line
-	2050 1800 2050 1950
-Wire Wire Line
-	2050 1650 2050 1750
-Connection ~ 2050 1800
-Wire Wire Line
-	2050 1750 2600 1750
 Wire Wire Line
 	2800 1750 2800 1650
-Connection ~ 2050 1750
-Wire Wire Line
-	2050 1750 2050 1800
-$Comp
-L power:+5V #PWR0115
-U 1 1 5C0D4464
-P 1350 1250
-AR Path="/5C0BBB2B/5C0D4464" Ref="#PWR0115"  Part="1"
-AR Path="/5C0BFA48/5C0D4464" Ref="#PWR?"  Part="1"
-F 0 "#PWR0115" H 1350 1100 50  0001 C CNN
-F 1 "+5V" H 1365 1423 50  0000 C CNN
-F 2 "" H 1350 1250 50  0001 C CNN
-F 3 "" H 1350 1250 50  0001 C CNN
-	1    1350 1250
-	1    0    0    -1
-$EndComp
-Wire Wire Line
-	1350 1250 1350 1350
 Wire Wire Line
 	1350 1350 1750 1350
@@
 Wire Wire Line
 	1350 1350 1350 1450
-Wire Wire Line
-	2800 1250 2800 1300
 Wire Wire Line
 	2350 1350 2600 1350
@@
 Wire Wire Line
 	2600 1650 2600 1750
-Connection ~ 2600 1750
-Wire Wire Line
-	2600 1750 2800 1750
+Wire Wire Line
+	2600 1750 2700 1750
 $Comp
 L taobao-cp:CP47uf,50V C9
@@
 L Connector_Generic:Conn_01x03 J5
 U 1 1 5C078669
-P 3750 1650
+P 4450 1300
 AR Path="/5C0BBB2B/5C078669" Ref="J5"  Part="1"
 AR Path="/5C0BFA48/5C078669" Ref="J?"  Part="1"
-F 0 "J5" H 3670 1967 50  0000 C CNN
-F 1 "Conn_01x03" H 3670 1876 50  0000 C CNN
-F 2 "Connector_PinHeader_2.54mm:PinHeader_1x03_P2.54mm_Vertical" H 3750 1650 50  0001 C CNN
-F 3 "~" H 3750 1650 50  0001 C CNN
-	1    3750 1650
-	-1   0    0    -1
+F 0 "J5" H 4370 1617 50  0000 C CNN
+F 1 "Conn_01x03" H 4370 1526 50  0000 C CNN
+F 2 "Connector_PinHeader_2.54mm:PinHeader_1x03_P2.54mm_Vertical" H 4450 1300 50  0001 C CNN
+F 3 "~" H 4450 1300 50  0001 C CNN
+	1    4450 1300
+	1    0    0    -1
 $EndComp
 $Comp
 L power:GND #PWR0116
 U 1 1 5C07899D
-P 4150 1400
+P 4050 1050
 AR Path="/5C0BBB2B/5C07899D" Ref="#PWR0116"  Part="1"
 AR Path="/5C0BFA48/5C07899D" Ref="#PWR?"  Part="1"
-F 0 "#PWR0116" H 4150 1150 50  0001 C CNN
-F 1 "GND" H 4155 1227 50  0000 C CNN
-F 2 "" H 4150 1400 50  0001 C CNN
-F 3 "" H 4150 1400 50  0001 C CNN
-	1    4150 1400
-	-1   0    0    1
-$EndComp
-Wire Wire Line
-	3950 1550 4150 1550
-Wire Wire Line
-	4150 1550 4150 1400
-Wire Wire Line
-	3950 1750 4150 1750
-Wire Wire Line
-	4150 1750 4150 1800
-Text Label 3350 1300 2    50   ~ 0
+F 0 "#PWR0116" H 4050 800 50  0001 C CNN
+F 1 "GND" H 4055 877 50  0000 C CNN
+F 2 "" H 4050 1050 50  0001 C CNN
+F 3 "" H 4050 1050 50  0001 C CNN
+	1    4050 1050
+	1    0    0    1
+$EndComp
+Wire Wire Line
+	4250 1200 4050 1200
+Wire Wire Line
+	4050 1200 4050 1050
+Wire Wire Line
+	4250 1400 4050 1400
+Wire Wire Line
+	4050 1400 4050 1450
+Text Label 3350 950  2    50   ~ 0
 OUTPUT
 Wire Wire Line
-	2800 1300 3350 1300
-Connection ~ 2800 1300
-Wire Wire Line
-	2800 1300 2800 1350
-Text Label 4500 1650 2    50   ~ 0
+	2800 950  3350 950
+Text Label 3700 1300 0    50   ~ 0
 OUTPUT
 Wire Wire Line
-	3950 1650 4500 1650
+	4250 1300 3700 1300
 $Comp
 L power:+3V3 #PWR0117
 U 1 1 5C0C0902
-P 2800 1250
-F 0 "#PWR0117" H 2800 1100 50  0001 C CNN
-F 1 "+3V3" H 2850 1450 50  0000 C CNN
-F 2 "" H 2800 1250 50  0001 C CNN
-F 3 "" H 2800 1250 50  0001 C CNN
-	1    2800 1250
+P 2800 900
+F 0 "#PWR0117" H 2800 750 50  0001 C CNN
+F 1 "+3V3" H 2850 1100 50  0000 C CNN
+F 2 "" H 2800 900 50  0001 C CNN
+F 3 "" H 2800 900 50  0001 C CNN
+	1    2800 900
 	1    0    0    -1
 $EndComp
@@
 L power:+3V3 #PWR0118
 U 1 1 5C0C0B31
-P 4150 1800
-F 0 "#PWR0118" H 4150 1650 50  0001 C CNN
-F 1 "+3V3" H 4150 2000 50  0000 C CNN
-F 2 "" H 4150 1800 50  0001 C CNN
-F 3 "" H 4150 1800 50  0001 C CNN
-	1    4150 1800
-	-1   0    0    1
+P 4050 1450
+F 0 "#PWR0118" H 4050 1300 50  0001 C CNN
+F 1 "+3V3" H 4050 1650 50  0000 C CNN
+F 2 "" H 4050 1450 50  0001 C CNN
+F 3 "" H 4050 1450 50  0001 C CNN
+	1    4050 1450
+	1    0    0    1
 $EndComp
 $Comp
@@
 	0    -1   -1   0
 $EndComp
+$Comp
+L taobao-components:VIN #PWR?
+U 1 1 5C1480E5
+P 1350 950
+F 0 "#PWR?" H 1350 800 50  0001 C CNN
+F 1 "VIN" H 1400 1100 50  0000 C CNN
+F 2 "" H 1350 950 50  0001 C CNN
+F 3 "" H 1350 950 50  0001 C CNN
+	1    1350 950
+	1    0    0    -1
+$EndComp
+$Comp
+L Device:Jumper_NO_Small JP?
+U 1 1 5C148323
+P 1350 1100
+F 0 "JP?" V 1300 1150 50  0000 L CNN
+F 1 "Jumper_NO_Small" V 1350 1150 50  0000 L CNN
+F 2 "" H 1350 1100 50  0001 C CNN
+F 3 "~" H 1350 1100 50  0001 C CNN
+	1    1350 1100
+	0    1    1    0
+$EndComp
+Wire Wire Line
+	1350 950  1350 1000
+Wire Wire Line
+	1350 1200 1350 1350
+$Comp
+L Device:Jumper_NO_Small JP?
+U 1 1 5C148F3B
+P 2800 1100
+F 0 "JP?" V 2750 1150 50  0000 L CNN
+F 1 "Jumper_NO_Small" V 2800 1150 50  0000 L CNN
+F 2 "" H 2800 1100 50  0001 C CNN
+F 3 "~" H 2800 1100 50  0001 C CNN
+	1    2800 1100
+	0    1    1    0
+$EndComp
+Wire Wire Line
+	2800 950  2800 1000
+Connection ~ 2800 950
+Wire Wire Line
+	2800 1200 2800 1350
+Wire Wire Line
+	2800 900  2800 950
+Wire Wire Line
+	2050 1650 2050 1950
+$Comp
+L power:GND #PWR?
+U 1 1 5C14BD92
+P 2700 1950
+AR Path="/5C0BBB2B/5C14BD92" Ref="#PWR?"  Part="1"
+AR Path="/5C0BFA48/5C14BD92" Ref="#PWR?"  Part="1"
+F 0 "#PWR?" H 2700 1700 50  0001 C CNN
+F 1 "GND" H 2750 1750 50  0000 C CNN
+F 2 "" H 2700 1950 50  0001 C CNN
+F 3 "" H 2700 1950 50  0001 C CNN
+	1    2700 1950
+	1    0    0    -1
+$EndComp
+Wire Wire Line
+	2700 1750 2700 1950
+Connection ~ 2700 1750
+Wire Wire Line
+	2700 1750 2800 1750
+$Comp
+L power:GND #PWR?
+U 1 1 5C14C0B1
+P 1350 1950
+AR Path="/5C0BBB2B/5C14C0B1" Ref="#PWR?"  Part="1"
+AR Path="/5C0BFA48/5C14C0B1" Ref="#PWR?"  Part="1"
+F 0 "#PWR?" H 1350 1700 50  0001 C CNN
+F 1 "GND" H 1400 1750 50  0000 C CNN
+F 2 "" H 1350 1950 50  0001 C CNN
+F 3 "" H 1350 1950 50  0001 C CNN
+	1    1350 1950
+	1    0    0    -1
+$EndComp
+Wire Wire Line
+	1350 1650 1350 1950
 $EndSCHEMATC

Commit message: update,
Connections:
- net VIN renamed +5V
Changed lines of the file:
@@
-$EndComp
-$Comp
-L taobao-components:VIN #PWR?
-U 1 1 5C1480E5
-P 1350 950
-F 0 "#PWR?" H 1350 800 50  0001 C CNN
-F 1 "VIN" H 1400 1100 50  0000 C CNN
-F 2 "" H 1350 950 50  0001 C CNN
-F 3 "" H 1350 950 50  0001 C CNN
-	1    1350 950
-	1    0    0    -1
 $EndComp
 $Comp
@@
 Wire Wire Line
 	1350 1650 1350 1950
+$Comp
+L power:+5V #PWR?
+U 1 1 5C153651
+P 1350 950
+F 0 "#PWR?" H 1350 800 50  0001 C CNN
+F 1 "+5V" H 1400 1150 50  0000 C CNN
+F 2 "" H 1350 950 50  0001 C CNN
+F 3 "" H 1350 950 50  0001 C CNN
+	1    1350 950
+	1    0    0    -1
+$EndComp
 $EndSCHEMATC

Commit message: update,
Parts:
- gave numbers to parts that had none: 2
Changed lines of the file:
@@
 $EndComp
 $Comp
-L Device:Jumper_NO_Small JP?
+L Device:Jumper_NO_Small JP2
 U 1 1 5C148323
 P 1350 1100
-F 0 "JP?" V 1300 1150 50  0000 L CNN
+F 0 "JP2" V 1300 1150 50  0000 L CNN
 F 1 "Jumper_NO_Small" V 1350 1150 50  0000 L CNN
 F 2 "" H 1350 1100 50  0001 C CNN
@@
 	1350 1200 1350 1350
 $Comp
-L Device:Jumper_NO_Small JP?
+L Device:Jumper_NO_Small JP3
 U 1 1 5C148F3B
 P 2800 1100
-F 0 "JP?" V 2750 1150 50  0000 L CNN
+F 0 "JP3" V 2750 1150 50  0000 L CNN
 F 1 "Jumper_NO_Small" V 2800 1150 50  0000 L CNN
 F 2 "" H 2800 1100 50  0001 C CNN
@@
 	2050 1650 2050 1950
 $Comp
-L power:GND #PWR?
+L power:GND #PWR0137
 U 1 1 5C14BD92
 P 2700 1950
-AR Path="/5C0BBB2B/5C14BD92" Ref="#PWR?"  Part="1"
+AR Path="/5C0BBB2B/5C14BD92" Ref="#PWR0137"  Part="1"
 AR Path="/5C0BFA48/5C14BD92" Ref="#PWR?"  Part="1"
-F 0 "#PWR?" H 2700 1700 50  0001 C CNN
+F 0 "#PWR0137" H 2700 1700 50  0001 C CNN
 F 1 "GND" H 2750 1750 50  0000 C CNN
 F 2 "" H 2700 1950 50  0001 C CNN
@@
 	2700 1750 2800 1750
 $Comp
-L power:GND #PWR?
+L power:GND #PWR0138
 U 1 1 5C14C0B1
 P 1350 1950
-AR Path="/5C0BBB2B/5C14C0B1" Ref="#PWR?"  Part="1"
+AR Path="/5C0BBB2B/5C14C0B1" Ref="#PWR0138"  Part="1"
 AR Path="/5C0BFA48/5C14C0B1" Ref="#PWR?"  Part="1"
-F 0 "#PWR?" H 1350 1700 50  0001 C CNN
+F 0 "#PWR0138" H 1350 1700 50  0001 C CNN
 F 1 "GND" H 1400 1750 50  0000 C CNN
 F 2 "" H 1350 1950 50  0001 C CNN
@@
 	1350 1650 1350 1950
 $Comp
-L power:+5V #PWR?
+L power:+5V #PWR0139
 U 1 1 5C153651
 P 1350 950
-F 0 "#PWR?" H 1350 800 50  0001 C CNN
+F 0 "#PWR0139" H 1350 800 50  0001 C CNN
 F 1 "+5V" H 1400 1150 50  0000 C CNN
 F 2 "" H 1350 950 50  0001 C CNN
