File: ATMEGA328P.sch (KiCad schematic (older format))
At the start: 16 parts, among them J1 Conn_01x08, J2 Conn_01x06, J3 Conn_01x06, J4 Conn_01x08, SW1 SW_Push, U1 ATMEGA328P, Y1 O16M

Commit message: update,
Parts:
- removed C2: C104,0603, Capacitor_SMD:C_0603_1608Metric_Pad1.05x0.95mm_HandSolder, symbol taobao-c:C104,0603
- removed R1: R104,0603, Resistor_SMD:R_0603_1608Metric_Pad1.05x0.95mm_HandSolder, symbol taobao-r:R104,0603
- removed SW1: SW_Push, Button_Switch_SMD:SW_SPST_CK_RS282G05A3, symbol Switch:SW_Push
- added C?: C104,0603, Capacitor_SMD:C_0603_1608Metric_Pad1.05x0.95mm_HandSolder, symbol taobao-c:C104,0603
- added R?: R104,0603, Resistor_SMD:R_0603_1608Metric_Pad1.05x0.95mm_HandSolder, symbol taobao-r:R104,0603
- added SW?: SW_Push, Button_Switch_SMD:SW_SPST_CK_RS282G05A3, symbol Switch:SW_Push
Connections:
- net GND: now also C?.2, SW?.1
- net RESET: now also C?.1, R?.2, SW?.2
- net Vio: now also R?.1

Commit message: update,
Changed lines of the file:
@@
 $EndComp
-Wire Wire Line
-	5250 4950 5250 4750
-Wire Wire Line
-	5250 3900 5500 3900
 Wire Wire Line
 	5500 4350 5250 4350
-Connection ~ 5250 4350
-Wire Wire Line
-	5250 4350 5250 3900
 $Comp
 L taobao-c:C104,0603 C6
@@
 Wire Wire Line
 	4900 4250 4900 4300
-Wire Wire Line
-	4900 4500 4900 4750
-Wire Wire Line
-	4900 4750 5250 4750
-Connection ~ 5250 4750
-Wire Wire Line
-	5250 4750 5250 4350
 $Comp
 L taobao-osc:O16M Y1
@@
 	4500 3800 4500 3900
 Connection ~ 4500 3800
-Wire Wire Line
-	4500 4500 4500 4750
-Wire Wire Line
-	4500 4750 4900 4750
-Connection ~ 4900 4750
 Wire Wire Line
 	5050 3700 5500 3700
@@
 EndData
 $EndBitmap
+Wire Wire Line
+	5250 4350 5250 4950
+$Comp
+L power:GND #PWR?
+U 1 1 5C118F23
+P 4900 4950
+AR Path="/5C08084B/5C118F23" Ref="#PWR?"  Part="1"
+AR Path="/5C0BBB2B/5C118F23" Ref="#PWR?"  Part="1"
+F 0 "#PWR?" H 4900 4700 50  0001 C CNN
+F 1 "GND" H 4950 4750 50  0000 C CNN
+F 2 "" H 4900 4950 50  0001 C CNN
+F 3 "" H 4900 4950 50  0001 C CNN
+	1    4900 4950
+	1    0    0    -1
+$EndComp
+$Comp
+L power:GND #PWR?
+U 1 1 5C118F4E
+P 4500 4950
+AR Path="/5C08084B/5C118F4E" Ref="#PWR?"  Part="1"
+AR Path="/5C0BBB2B/5C118F4E" Ref="#PWR?"  Part="1"
+F 0 "#PWR?" H 4500 4700 50  0001 C CNN
+F 1 "GND" H 4550 4750 50  0000 C CNN
+F 2 "" H 4500 4950 50  0001 C CNN
+F 3 "" H 4500 4950 50  0001 C CNN
+	1    4500 4950
+	1    0    0    -1
+$EndComp
+Wire Wire Line
+	4500 4500 4500 4950
+Wire Wire Line
+	4900 4500 4900 4950
+$Comp
+L power:GND #PWR?
+U 1 1 5C11E3A6
+P 4700 4950
+AR Path="/5C08084B/5C11E3A6" Ref="#PWR?"  Part="1"
+AR Path="/5C0BBB2B/5C11E3A6" Ref="#PWR?"  Part="1"
+F 0 "#PWR?" H 4700 4700 50  0001 C CNN
+F 1 "GND" H 4750 4750 50  0000 C CNN
+F 2 "" H 4700 4950 50  0001 C CNN
+F 3 "" H 4700 4950 50  0001 C CNN
+	1    4700 4950
+	1    0    0    -1
+$EndComp
+Wire Wire Line
+	4700 4950 4700 3900
+Wire Wire Line
+	4700 3900 5500 3900
 $EndSCHEMATC

Commit message: update,
Parts:
- gave numbers to parts that had none: 3
Changed lines of the file:
@@
 	2600 4100 2450 4100
 $Comp
-L Switch:SW_Push SW?
+L Switch:SW_Push SW1
 U 1 1 5C1691AC
 P 4500 1800
-AR Path="/5C08084B/5C1691AC" Ref="SW?"  Part="1"
+AR Path="/5C08084B/5C1691AC" Ref="SW1"  Part="1"
 AR Path="/5C0BBB2B/5C1691AC" Ref="SW?"  Part="1"
-F 0 "SW?" H 4500 2100 50  0000 C CNN
+F 0 "SW1" H 4500 2100 50  0000 C CNN
 F 1 "SW_Push" H 4500 2000 50  0000 C CNN
 F 2 "Button_Switch_SMD:SW_SPST_CK_RS282G05A3" H 4500 2000 50  0001 C CNN
@@
 $EndComp
 $Comp
-L taobao-c:C104,0603 C?
+L taobao-c:C104,0603 C2
 U 1 1 5C16924D
 P 5000 1800
-AR Path="/5C08084B/5C16924D" Ref="C?"  Part="1"
+AR Path="/5C08084B/5C16924D" Ref="C2"  Part="1"
 AR Path="/5C0BBB2B/5C16924D" Ref="C?"  Part="1"
-F 0 "C?" H 5100 1850 50  0000 L CNN
+F 0 "C2" H 5100 1850 50  0000 L CNN
 F 1 "C104,0603" H 5100 1800 50  0000 L CNN
 F 2 "Capacitor_SMD:C_0603_1608Metric_Pad1.05x0.95mm_HandSolder" H 5000 1800 50  0001 C CNN
@@
 $EndComp
 $Comp
-L taobao-r:R104,0603 R?
+L taobao-r:R104,0603 R1
 U 1 1 5C1692A3
 P 5000 1300
-AR Path="/5C08084B/5C1692A3" Ref="R?"  Part="1"
+AR Path="/5C08084B/5C1692A3" Ref="R1"  Part="1"
 AR Path="/5C0BBB2B/5C1692A3" Ref="R?"  Part="1"
-F 0 "R?" H 5100 1350 50  0000 L CNN
+F 0 "R1" H 5100 1350 50  0000 L CNN
 F 1 "R104,0603" H 5100 1300 50  0000 L CNN
 F 2 "Resistor_SMD:R_0603_1608Metric_Pad1.05x0.95mm_HandSolder" H 5000 1300 50  0001 C CNN
@@
 $EndComp
 $Comp
-L taobao-components:Vio #PWR?
+L taobao-components:Vio #PWR0107
 U 1 1 5C16931D
 P 5000 850
-AR Path="/5C08084B/5C16931D" Ref="#PWR?"  Part="1"
+AR Path="/5C08084B/5C16931D" Ref="#PWR0107"  Part="1"
 AR Path="/5C0BBB2B/5C16931D" Ref="#PWR?"  Part="1"
-F 0 "#PWR?" H 5000 700 50  0001 C CNN
+F 0 "#PWR0107" H 5000 700 50  0001 C CNN
 F 1 "Vio" H 5050 1000 50  0000 C CNN
 F 2 "" H 5000 850 50  0001 C CNN
@@
 	5000 1500 5000 1600
 $Comp
-L power:GND #PWR?
+L power:GND #PWR0108
 U 1 1 5C173027
 P 4500 2150
-F 0 "#PWR?" H 4500 1900 50  0001 C CNN
+F 0 "#PWR0108" H 4500 1900 50  0001 C CNN
 F 1 "GND" H 4550 1950 50  0000 C CNN
 F 2 "" H 4500 2150 50  0001 C CNN
@@
 $EndComp
 $Comp
-L power:GND #PWR?
+L power:GND #PWR0115
 U 1 1 5C17305F
 P 5000 2150
-F 0 "#PWR?" H 5000 1900 50  0001 C CNN
+F 0 "#PWR0115" H 5000 1900 50  0001 C CNN
 F 1 "GND" H 5050 1950 50  0000 C CNN
 F 2 "" H 5000 2150 50  0001 C CNN
@@
 	5250 4350 5250 4950
 $Comp
-L power:GND #PWR?
+L power:GND #PWR0128
 U 1 1 5C118F23
 P 4900 4950
-AR Path="/5C08084B/5C118F23" Ref="#PWR?"  Part="1"
+AR Path="/5C08084B/5C118F23" Ref="#PWR0128"  Part="1"
 AR Path="/5C0BBB2B/5C118F23" Ref="#PWR?"  Part="1"
-F 0 "#PWR?" H 4900 4700 50  0001 C CNN
+F 0 "#PWR0128" H 4900 4700 50  0001 C CNN
 F 1 "GND" H 4950 4750 50  0000 C CNN
 F 2 "" H 4900 4950 50  0001 C CNN
@@
 $EndComp
 $Comp
-L power:GND #PWR?
+L power:GND #PWR0129
 U 1 1 5C118F4E
 P 4500 4950
-AR Path="/5C08084B/5C118F4E" Ref="#PWR?"  Part="1"
+AR Path="/5C08084B/5C118F4E" Ref="#PWR0129"  Part="1"
 AR Path="/5C0BBB2B/5C118F4E" Ref="#PWR?"  Part="1"
-F 0 "#PWR?" H 4500 4700 50  0001 C CNN
+F 0 "#PWR0129" H 4500 4700 50  0001 C CNN
 F 1 "GND" H 4550 4750 50  0000 C CNN
 F 2 "" H 4500 4950 50  0001 C CNN
@@
 	4900 4500 4900 4950
 $Comp
-L power:GND #PWR?
+L power:GND #PWR0136
 U 1 1 5C11E3A6
 P 4700 4950
-AR Path="/5C08084B/5C11E3A6" Ref="#PWR?"  Part="1"
+AR Path="/5C08084B/5C11E3A6" Ref="#PWR0136"  Part="1"
 AR Path="/5C0BBB2B/5C11E3A6" Ref="#PWR?"  Part="1"
-F 0 "#PWR?" H 4700 4700 50  0001 C CNN
+F 0 "#PWR0136" H 4700 4700 50  0001 C CNN
 F 1 "GND" H 4750 4750 50  0000 C CNN
 F 2 "" H 4700 4950 50  0001 C CNN

Commit message: update,
Parts:
- removed C1: C104,0603, Capacitor_SMD:C_0603_1608Metric_Pad1.05x0.95mm_HandSolder, symbol taobao-c:C104,0603
- removed J1: Conn_01x08, Connector_PinHeader_2.54mm:PinHeader_1x08_P2.54mm_Vertical, symbol Connector_Generic:Conn_01x08
- removed J2, J3: Conn_01x06, Connector_PinHeader_2.54mm:PinHeader_1x06_P2.54mm_Vertical, symbol Connector_Generic:Conn_01x06
- removed JP1: Jumper_3_Bridged12, Connector_PinHeader_2.00mm:PinHeader_1x03_P2.00mm_Vertical, symbol Jumper:Jumper_3_Bridged12
- removed U1: ATMEGA328P, Package_QFP:TQFP-32_7x7mm_P0.8mm, symbol taobao-components:ATMEGA328P
- added C1: C106,0603, Capacitor_SMD:C_0603_1608Metric_Pad1.05x0.95mm_HandSolder, symbol taobao-c:C106,0603
- added C13: C104,0603, Capacitor_SMD:C_0603_1608Metric_Pad1.05x0.95mm_HandSolder, symbol taobao-c:C104,0603
- added C14: C105,0603, Capacitor_SMD:C_0603_1608Metric_Pad1.05x0.95mm_HandSolder, symbol taobao-c:C105,0603
- added D3: LED_GREEN,0603, LED_SMD:LED_0603_1608Metric_Pad1.05x0.95mm_HandSolder, symbol taobao-led:LED_GREEN,0603
- added J1: Conn_01x02, Connector_PinHeader_1.27mm:PinHeader_1x02_P1.27mm_Vertical, symbol Connector_Generic:Conn_01x02
- added R5: R103,0603, Resistor_SMD:R_0603_1608Metric_Pad1.05x0.95mm_HandSolder, symbol taobao-r:R103,0603
- added U1: ATMEGA328P-TQFP, Package_QFP:TQFP-32_7x7mm_P0.8mm, symbol taobao-components:ATMEGA328P-TQFP
- added U4: CONN_ARDUINO_ICSP, Connector_PinHeader_2.54mm:PinHeader_2x03_P2.54mm_Vertical, symbol taobao-components:CONN_ARDUINO_ICSP
- J4: value Conn_01x08 -> Conn_01x02; footprint Connector_PinHeader_2.54mm:PinHeader_1x08_P2.54mm_Vertical -> Connector_PinHeader_2.54mm:PinHeader_1x02_P2.54mm_Vertical; symbol Connector_Generic:Conn_01x08 -> Connector_Generic:Conn_01x02
Connections:
- net labels added: MISO, MOSI, SCK, VCC
- net labels removed: +3V3, AREF, VBUS, VCCIO, VIN, Vio
- wire segments 88 -> 87
Other:
- moved on the sheet: C2, C3, C4, R1, R2, SW1, Y1
