File: ATMEGA328P_tryout.kicad_pcb (KiCad board)
At the start: 2 copper layers, 115 x 95 mm, 38 parts, among them J1 Conn_01x08, J2 Conn_01x06, J3 Conn_01x06, J4 Conn_01x08, J5 Conn_01x03, J6 Conn_01x03, J7 USB_B_Mini, SW1 SW_Push, U1 ATMEGA328P, U2 AMS1117-3.3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

Commit message: update,
Routing:
- net GND: track 0.00 -> 280.2 mm, vias 0 -> 1
- net +5V: track 0.00 -> 187.7 mm, vias 0 -> 1
- net VIN: track 0.00 -> 115.8 mm
- net +3V3: track 0.00 -> 77.1 mm
- net VCCIO: track 0.00 -> 63.3 mm, vias 0 -> 2
- net RESET: track 0.00 -> 59.6 mm, vias 0 -> 1
- net TXD: track 0.00 -> 53.9 mm, vias 0 -> 1
- net RXD: track 0.00 -> 45.9 mm
- net DTR: track 0.00 -> 30.9 mm
- net Net-(J3-Pad6): track 0.00 -> 28.9 mm
- net Net-(J4-Pad8): track 0.00 -> 28.6 mm
- net Net-(J4-Pad1): track 0.00 -> 28.4 mm
- net Net-(J3-Pad5): track 0.00 -> 27.1 mm
- net Net-(J4-Pad2): track 0.00 -> 26.8 mm
- net Net-(J4-Pad3): track 0.00 -> 26.7 mm
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
Commit message: update,
Parts:
- moved C6 36.7 mm to (84.6, 81.7), turned to 90 degrees
- moved C1 7.11 mm to (51.3, 41.6)
- moved D5 5.63 mm to (39.5, 59.2), turned to 0 degrees
- moved R1 4.10 mm to (80.6, 65.5)
- moved C5 0.32 mm to (100.2, 83.8)
- turned D3 to 270 degrees
- turned D4 to 270 degrees
Routing:
- net RESET: track 59.6 -> 71.4 mm
- net VIN: track 115.8 -> 124.5 mm
- net +5V: track 187.7 -> 194.8 mm
- net GND: track 280.2 -> 275.8 mm, vias 1 -> 3
- net RXD: track 45.9 -> 49.9 mm
- net DTR: track 30.9 -> 33.6 mm
- net TXD: track 53.9 -> 56.5 mm
- net VCCIO: track 63.3 -> 60.8 mm
- net Net-(C3-Pad1): track 13.7 -> 15.9 mm
- net Net-(D5-Pad2): track 8.01 -> 6.14 mm
- net Net-(J7-Pad3): track 10.3 -> 11.9 mm
- net Net-(C4-Pad1): track 13.9 -> 15.3 mm
- net Net-(R6-Pad2): track 4.90 -> 5.84 mm
- net Net-(D4-Pad1): track 1.67 -> 2.44 mm
- net Net-(D3-Pad1): track 2.00 -> 2.72 mm

Commit message: update,
Parts:
- added J8: USB_B_Mini, Connector_USB:USB_Micro-B_Amphenol_10103594-0001LF_Horizontal, F.Cu at (36.1, 41.5)
- J7: value USB_B_Mini -> Conn_01x02
Connections:
- C10 pad 1: VIN -> Net-(C10-Pad1)
- C11 pad 1: +5V -> Net-(C11-Pad1)
- C12 pad 1: +5V -> Net-(C11-Pad1)
- C2 pad 2: DTR -> GND
- C7 pad 1: +5V -> Net-(C7-Pad1)
- C8 pad 1: +3V3 -> Net-(C8-Pad1)
- C9 pad 1: +3V3 -> Net-(C8-Pad1)
- J7 pad 1: Net-(D5-Pad2) -> GND
- J7 pad 2: Net-(J7-Pad2) -> VIN
- J7 pad 3: Net-(J7-Pad3) -> (no net)
- J7 pad 4: Net-(J7-Pad4) -> (no net)
- J7 pad 5: GND -> (no net)
- J7 pad 6: GND -> (no net)
- U2 pad 2: +3V3 -> Net-(C8-Pad1)
- U2 pad 3: +5V -> Net-(C7-Pad1)
- U3 pad 2: +5V -> Net-(C11-Pad1)
- U3 pad 3: VIN -> Net-(C10-Pad1)
- U4 pad 3: Net-(J7-Pad3) -> D_P
- U4 pad 4: Net-(J7-Pad2) -> D_M
- U4 pad 5: Net-(U4-Pad5) -> +3V3
- U4 pad 6: Net-(U4-Pad5) -> +3V3
- U4 pad 7: Net-(U4-Pad5) -> +3V3
Routing:
- net +3V3: track 77.1 -> 78.6 mm
- net Net-(U4-Pad5): track 1.53 -> 0.00 mm

Commit message: update,
Parts:
- removed C10, C11, C7, C8: C104,0603, Capacitor_SMD:C_0603_1608Metric_Pad1.05x0.95mm_HandSolder
- removed C12, C9: CP47uf,50V, w_smd_cap:c_elec_6.3x7.7
- removed D1, D2: LED_GREEN,0603, LED_SMD:LED_0603_1608Metric_Pad1.05x0.95mm_HandSolder
- removed D4: LED_ORANGE,0603, LED_SMD:LED_0603_1608Metric_Pad1.05x0.95mm_HandSolder
- removed D5: SD_1N4001_M1, w_smd_diode:do214ac
- removed J2, J3: Conn_01x06, Connector_PinHeader_2.54mm:PinHeader_1x06_P2.54mm_Vertical
- removed J5, J6: Conn_01x03, Connector_PinHeader_2.54mm:PinHeader_1x03_P2.54mm_Vertical
- removed J7: Conn_01x02, Connector_USB:USB_Micro-B_Amphenol_10103594-0001LF_Horizontal
- removed J8: USB_B_Mini, Connector_USB:USB_Micro-B_Amphenol_10103594-0001LF_Horizontal
- removed JP1: Jumper_3_Bridged12, Connector_PinHeader_2.00mm:PinHeader_1x03_P2.00mm_Vertical
- removed R3, R4, R6: R102,0603, Resistor_SMD:R_0603_1608Metric_Pad1.05x0.95mm_HandSolder
- removed U2: AMS1117-3.3, Package_TO_SOT_SMD:SOT-223-3_TabPin2
- removed U3: AMS1117-5.0, Package_TO_SOT_SMD:SOT-223-3_TabPin2
- added C14: C105,0603, Capacitor_SMD:C_0603_1608Metric_Pad1.05x0.95mm_HandSolder, B.Cu at (37.3, 41.9)
- C1: value C104,0603 -> C106,0603
- C13: value C106,0603 -> C104,0603; moved to B.Cu
- C2, C3, C4, C5, C6, R2: moved to B.Cu
- D3: value LED_ORANGE,0603 -> LED_GREEN,0603
- J1: value Conn_01x08 -> Conn_01x02; footprint Connector_PinHeader_2.54mm:PinHeader_1x08_P2.54mm_Vertical -> Connector_PinHeader_1.27mm:PinHeader_1x02_P1.27mm_Vertical
- J4: value Conn_01x08 -> Conn_01x02; footprint Connector_PinHeader_2.54mm:PinHeader_1x08_P2.54mm_Vertical -> Connector_PinHeader_2.54mm:PinHeader_1x02_P2.54mm_Vertical
- R5: value R102,0603 -> R103,0603; moved to B.Cu
- U1: value ATMEGA328P -> ATMEGA328P-TQFP
- U4: value CP2104 -> CONN_ARDUINO_ICSP; footprint Package_DFN_QFN:QFN-24-1EP_4x4mm_P0.5mm_EP2.7x2.6mm_ThermalVias -> Connector_PinHeader_2.54mm:PinHeader_2x03_P2.54mm_Vertical
- moved C5 84.3 mm to (28.8, 39.1), turned to 0 degrees
- moved J4 76.6 mm to (32.2, 27.5), turned to 90 degrees
- moved C3 74.7 mm to (23.8, 36.6), turned to 270 degrees
- moved Y1 74.4 mm to (23.8, 38.5), turned to 270 degrees
- moved U1 73.9 mm to (33.0, 39.9)
- moved R2 71.5 mm to (31.8, 35.5), turned to 270 degrees
- moved C6 69.2 mm to (28.8, 40.7), turned to 0 degrees
- moved C4 69.2 mm to (23.8, 40.2), turned to 90 degrees
- moved C2 56.3 mm to (33.5, 31.6), turned to 180 degrees
- moved SW1 54.6 mm to (33.5, 31.6), turned to 0 degrees
- moved R1 50.7 mm to (39.2, 36.2), turned to 90 degrees
- moved R5 47.4 mm to (27.5, 31.5)
- moved D3 46.3 mm to (27.5, 31.5)
- moved U4 34.7 mm to (42.0, 31.0)
- moved C13 31.0 mm to (37.3, 39.9), turned to 180 degrees
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Connections:
- C1 pad 1: Net-(C1-Pad1) -> GND
- C1 pad 2: GND -> VCC
- C2 pad 1: RESET -> /ATMEGA328P/RESET
- C5 pad 1: VCCIO -> VCC
- C6 pad 1: VCCIO -> VCC
- D3 pad 1: Net-(D3-Pad1) -> GND
- D3 pad 2: +5V -> Net-(D3-Pad2)
- J1 pad 1: VBUS -> +5V
- J1 pad 2: RESET -> VCC
- J4 pad 1: Net-(J4-Pad1) -> TXD
- R1 pad 1: VCCIO -> VCC
- R1 pad 2: RESET -> /ATMEGA328P/RESET
- R2 pad 1: Net-(J4-Pad8) -> RXD
- R2 pad 2: RXD -> Net-(J4-Pad2)
- R5 pad 1: Net-(D3-Pad1) -> Net-(D3-Pad2)
- R5 pad 2: Net-(R5-Pad2) -> VCC
- SW1 pad 2: RESET -> /ATMEGA328P/RESET
- U1 pad 1: Net-(J4-Pad5) -> Net-(U1-Pad1)
- U1 pad 10: Net-(J4-Pad2) -> Net-(U1-Pad10)
- U1 pad 11: Net-(J4-Pad1) -> Net-(U1-Pad11)
- U1 pad 15: Net-(J2-Pad4) -> /ATMEGA328P/MOSI
- U1 pad 16: Net-(J2-Pad5) -> /ATMEGA328P/MISO
- U1 pad 17: Net-(J2-Pad6) -> /ATMEGA328P/SCK
- U1 pad 18: VCCIO -> VCC
- U1 pad 19: (no net) -> Net-(U1-Pad19)
- U1 pad 2: Net-(J4-Pad4) -> Net-(U1-Pad2)
- U1 pad 20: AREF -> Net-(C13-Pad1)
- U1 pad 22: (no net) -> Net-(U1-Pad22)
- U1 pad 29: RESET -> /ATMEGA328P/RESET
- U1 pad 30: Net-(J4-Pad8) -> Net-(J4-Pad2)
- U1 pad 32: Net-(J4-Pad6) -> Net-(U1-Pad32)
- U1 pad 4: VCCIO -> VCC
- U1 pad 5: (no net) -> GND
- U1 pad 6: (no net) -> VCC
- U1 pad 7: Net-(C4-Pad1) -> Net-(C3-Pad1)
- U1 pad 8: Net-(C3-Pad1) -> Net-(C4-Pad1)
- U1 pad 9: Net-(J4-Pad3) -> Net-(U1-Pad9)
- U4 pad 1: Net-(U4-Pad1) -> /ATMEGA328P/MISO
- U4 pad 2: GND -> VCC
- U4 pad 3: D_P -> /ATMEGA328P/SCK
- U4 pad 4: D_M -> /ATMEGA328P/MOSI
- U4 pad 5: +3V3 -> /ATMEGA328P/RESET
- U4 pad 6: +3V3 -> GND
Routing:
- net +5V: track 194.8 -> 0.00 mm, vias 1 -> 0
- net GND: track 275.8 -> 83.1 mm, vias 3 -> 0
- net VIN: track 124.5 -> 0.00 mm
- net +3V3: track 78.6 -> 0.00 mm
- net RESET: track 71.4 -> 0.00 mm, vias 1 -> 0
- net VCC: track 0.00 -> 65.8 mm
- net VCCIO: track 60.8 -> 0.00 mm, vias 2 -> 0
- net RXD: track 49.9 -> 0.00 mm
- net TXD: track 56.5 -> 8.65 mm, vias 1 -> 0
- net /ATMEGA328P/MOSI: track 0.00 -> 37.2 mm
- net DTR: track 33.6 -> 0.00 mm
- net Net-(U1-Pad28): track 28.9 -> 0.00 mm
- net Net-(J4-Pad8): track 28.6 -> 0.00 mm
- net Net-(J4-Pad1): track 28.4 -> 0.00 mm
- net Net-(U1-Pad27): track 27.1 -> 0.00 mm
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Other:
- board size 115 x 95 mm -> 30 x 25 mm
