File: ATMEGA328P_tryout.sch (KiCad schematic (older format))
At the start: 0 parts

Commit message: update,
Changed lines of the file:
@@
 $Descr A4 11693 8268
 encoding utf-8
-Sheet 1 5
+Sheet 1 2
 Title ""
 Date ""
@@
 F1 "ATMEGA328P.sch" 50
 $EndSheet
-$Sheet
-S 6150 5100 1200 800
-U 5C0BBB2B
-F0 "AMS1117-3.3_POWER_SUPPLY" 50
-F1 "AMS1117-3.3.sch" 50
-$EndSheet
-$Sheet
-S 6150 3500 1200 800
-U 5C0BFA48
-F0 "AMS1117-5V" 50
-F1 "AMS1117-5V.sch" 50
-$EndSheet
-$Sheet
-S 8100 3500 1200 800
-U 5C0C1365
-F0 "CP2104" 50
-F1 "CP2104.sch" 50
-$EndSheet
 $EndSCHEMATC
